File: hats/TFCB_ATV_TOP_HAT/TFCB_ATV_HAT.kicad_pcb (KiCad board)
At the start: 2 copper layers, 77.5 x 100 mm, 116 parts, among them J1 CONN_02X10, J10 Sense, J11 DISCRETE, J12 LID, J13 Analog OUT, J14 ISENSE, J2 CONN_02X10, J3 CONN_02X10, J4 CONN_02X10, J5 Power Input, J7 DISCHARGE, J8 WATCHDOG, J9 CN1, Q1 2N7002, Q10 2N7002, Q11 2N7002, Q12 2N7002, Q13 2N7002, Q14 2N7002, Q15 2N7002, Q16 2N7002, Q2 2N7002, Q3 2N7002, Q4 2N7002, Q5 2N7002, Q6 IRFS7437, Q7 IRFS7437, Q8 2N7002, Q9 2N7002, U1 TL082, U2 TL082, U3 TL082, U4 CD4040B, U5 TLE5012B, U6 TL082, U7 ADM4073, U8 PVG612

Commit message: More work on TFCB
Parts:
- added J6: 24V, bjh-kicad-connector-fp:Weidmuller-SL-5.08-Vertical-2Pole, F.Cu at (110.5, 54.7)
- added REF**: MountingHole_3-2mm, bjh-kicad-mountingholes-fp:MountingHole_3-2mm, F.Cu at (53.0, 53.0)
- added REF**: MountingHole_3-2mm, bjh-kicad-mountingholes-fp:MountingHole_3-2mm, F.Cu at (124.5, 53.0)
- added REF**: MountingHole_3-2mm, bjh-kicad-mountingholes-fp:MountingHole_3-2mm, F.Cu at (53.0, 147.0)
- added REF**: MountingHole_3-2mm, bjh-kicad-mountingholes-fp:MountingHole_3-2mm, F.Cu at (124.5, 147.0)
- C2, C4, C6, R11, R13, R14, R15, R16, R18, R2, R20, R22, R24, R25, R49, R5, R50, R52, R53, R8, U1, U5, U6, U7: moved to B.Cu
- D4, D5: footprint Diodes_SMD:Diode-SMC_Handsoldering -> bjh-kicad-rcld-fp:Diode_SMB
- J1, J2, J3, J4: footprint bjh-kicad-connector-fp:RCPT-2row-2.54mm-10way -> bjh-kicad-connector-fp:RCPT-2row-2.54mm-20way; moved to B.Cu
- J5: value Power Input -> POWER; footprint bjh-kicad-connector-fp:Weidmuller-SL-5.08-Vertical-5Pole -> bjh-kicad-connector-fp:Weidmuller-SL-5.08-Vertical-4Pole
- R37: footprint Resistors_SMD:R_0805_HandSoldering -> bjh-kicad-rcld-fp:PWR5322_SMD
- U4: footprint Housings_SOIC:SOIC-14_3.9x8.7mm_Pitch1.27mm -> Housings_SOIC:SOIC-16_3.9x9.9mm_Pitch1.27mm
- moved D6 198.8 mm to (83.3, 76.8), turned to 270 degrees
- moved R60 193.6 mm to (78.6, 80.0), turned to 180 degrees
- moved R61 190.6 mm to (86.5, 76.8), turned to 90 degrees
- moved C4 188.3 mm to (-13.5, 105.9), turned to 180 degrees
- moved R31 187.5 mm to (80.3, 105.9), turned to 180 degrees
- moved R5 187.5 mm to (-7.50, 103.1), turned to 180 degrees
- moved R26 181.7 mm to (77.7, 109.7), turned to 90 degrees
- moved R16 180.9 mm to (-13.5, 108.7), turned to 180 degrees
- moved R28 179.8 mm to (86.6, 110.9)
- moved R20 171.3 mm to (-18.2, 102.5), turned to 90 degrees
- moved R30 168.6 mm to (95.6, 109.1), turned to 270 degrees
- moved R22 167.0 mm to (-18.2, 97.4), turned to 270 degrees
- moved R8 165.8 mm to (-2.30, 102.5), turned to 90 degrees
- moved J1 165.7 mm to (73.5, 88.6), turned to 270 degrees
- moved C2 165.4 mm to (-7.49, 105.9)
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Connections:
- J1 pad 1: RH2 -> RH3
- J1 pad 10: RG4 -> ~MCLR
- J1 pad 2: RH3 -> RH2
- J1 pad 3: RE1 -> RE0
- J1 pad 4: RE0 -> RE1
- J1 pad 5: RG0 -> RG1
- J1 pad 6: RG1 -> RG0
- J1 pad 7: RG2 -> RG3
- J1 pad 8: RG3 -> RG2
- J1 pad 9: ~MCLR -> RG4
- J2 pad 1: RH5 -> RH4
- J2 pad 10: RA0 -> RA1
- J2 pad 2: RH4 -> RH5
- J2 pad 3: +3.3V -> GND
- J2 pad 4: GND -> +3.3V
- J2 pad 5: +3.3V -> GND
- J2 pad 6: GND -> +3.3V
- J2 pad 7: RA3 -> RA2
- J2 pad 8: RA2 -> RA3
- J2 pad 9: RA1 -> RA0
- J3 pad 1: RJ6 -> RJ7
- J3 pad 10: RA6 -> RA7
- J3 pad 2: RJ7 -> RJ6
- J3 pad 3: RC2 -> RC3
- J3 pad 4: RC3 -> RC2
- J3 pad 5: RC4 -> RC5
- J3 pad 6: RC5 -> RC4
- J3 pad 7: RB7 -> Net-(J3-Pad7)
- J3 pad 8: Net-(J3-Pad8) -> RB7
- J3 pad 9: RA7 -> RA6
- J4 pad 1: RJ1 -> RJ0
- J4 pad 10: GND -> RD1
- J4 pad 2: RJ0 -> RJ1
- J4 pad 3: RD7 -> RD6
- J4 pad 4: RD6 -> RD7
- J4 pad 5: RD5 -> RD4
- J4 pad 6: RD4 -> RD5
- J4 pad 7: RD3 -> RD2
- J4 pad 8: RD2 -> RD3
- J4 pad 9: RD1 -> GND
- J5 pad 1: GND -> +14V
- J5 pad 2: +3.3V -> +5V
- J5 pad 3: +5V -> +3.3V
- J5 pad 4: +14V -> GND
- Q10 pad 1: RE5 -> RJ7
- Q11 pad 1: RE3 -> RJ6
- Q5 pad 1: RE0 -> RJ3
- Q8 pad 1: RE4 -> RH5
- Q9 pad 1: RE2 -> RH4
- R33 pad 2: RE0 -> RJ3
- R40 pad 1: RE4 -> RH5
- R41 pad 1: RE5 -> RJ7
- R42 pad 1: RE2 -> RH4
- R43 pad 1: RE3 -> RJ6
- U3 pad 5: Net-(R49-Pad1) -> (no net)
- U3 pad 6: RA0 -> (no net)
- U3 pad 7: RA0 -> (no net)
- U4 pad 8: (no net) -> GND
- U6 pad 1: RA1 -> RA0
- U6 pad 2: RA1 -> RA0
- U6 pad 3: Net-(R50-Pad1) -> Net-(R49-Pad1)
- U6 pad 5: (no net) -> Net-(R50-Pad1)
- U6 pad 6: (no net) -> RA1
- U6 pad 7: (no net) -> RA1
Routing:
- net GND: track 0.00 -> 230.7 mm
- net +14V: track 0.00 -> 173.6 mm
- net +3.3V: track 0.00 -> 68.2 mm
- net CN1_5V: track 0.00 -> 43.6 mm
- net WDOG_OUT: track 0.00 -> 37.5 mm
- net J4-2: track 0.00 -> 35.8 mm
- net J4-1: track 0.00 -> 35.0 mm
- net J4-5: track 0.00 -> 32.8 mm
- net +5V: track 0.00 -> 29.3 mm
- net Net-(Q5-Pad3): track 0.00 -> 26.7 mm
- net RJ7: track 0.00 -> 26.1 mm
- net IFC: track 0.00 -> 23.2 mm
- net Net-(Q4-Pad1): track 0.00 -> 22.9 mm
- net RG0: track 0.00 -> 22.7 mm
- net Net-(Q9-Pad3): track 0.00 -> 22.6 mm
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Other:
- net class Default: trace_width 0.25 -> 0.4; via_dia 0.6 -> 1.27; via_drill 0.4 -> 0.8

Commit message: More work on the PCB layout
Parts:
- moved C2 71.3 mm to (63.7, 109.4)
- moved C4 71.3 mm to (57.7, 109.4)
- moved R11 71.3 mm to (68.9, 100.9)
- moved R16 71.3 mm to (57.6, 112.2)
- moved R18 71.3 mm to (57.7, 106.6)
- moved R2 71.3 mm to (63.7, 112.2)
- moved R20 71.3 mm to (53.0, 105.9)
- moved R22 71.3 mm to (53.0, 100.9)
- moved R5 71.3 mm to (63.7, 106.6)
- moved R8 71.3 mm to (68.9, 105.9)
- moved U1 71.3 mm to (60.7, 101.2)
- moved R9 13.8 mm to (53.0, 105.9), turned to 90 degrees
- moved R12 13.5 mm to (53.0, 100.9), turned to 270 degrees
- moved R3 12.1 mm to (57.6, 112.2), turned to 180 degrees
- moved R17 12.0 mm to (63.7, 112.2), turned to 0 degrees
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Routing:
- net RE7: track 0.00 -> 83.0 mm
- net RC2: track 0.00 -> 42.9 mm
- net Net-(R12-Pad1): track 4.67 -> 34.4 mm, vias 0 -> 1
- net Net-(R23-Pad1): track 4.77 -> 32.1 mm, vias 0 -> 1
- net Net-(R22-Pad1): track 5.45 -> 30.1 mm
- net RG0: track 22.7 -> 41.8 mm, vias 0 -> 1
- net RG3: track 11.6 -> 23.9 mm
- net GND: track 230.7 -> 242.4 mm
- net Net-(R11-Pad1): track 5.57 -> 16.3 mm
- net Net-(R10-Pad1): track 4.00 -> 12.7 mm, vias 0 -> 1
- net AO4: track 0.00 -> 7.03 mm
- net AO3: track 0.00 -> 7.03 mm
- net AO2: track 0.00 -> 7.03 mm
- net Net-(C3-Pad1): track 11.0 -> 5.62 mm
- net Net-(C5-Pad1): track 11.0 -> 5.66 mm
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
Commit message: More work to TFCB
Parts:
- D4, D5: value D -> D-BJH
- moved R51 15.3 mm to (73.2, 140.4), turned to 90 degrees
- moved R57 3.22 mm to (59.1, 141.4)
- moved D5 1.68 mm to (121.2, 138.2), turned to 90 degrees
- moved C6 1.31 mm to (112.8, 89.9)
- renumbered REF** to Mount1, REF** to Mount2, REF** to Mount3, REF** to Mount4
Connections:
- D4 pad A: (no net) -> Net-(D2-Pad2)
- D4 pad K: (no net) -> +5V
- D5 pad A: (no net) -> Net-(D3-Pad2)
- D5 pad K: (no net) -> +5V
- Q12 pad 1: RG1 -> RH6
- Q14 pad 1: RG2 -> RH7
- R48 pad 2: RG1 -> RH6
- R56 pad 2: RG2 -> RH7
Routing:
- net GND: track 242.4 -> 629.3 mm
- net +5V: track 29.3 -> 232.4 mm
- net +3.3V: track 68.2 -> 189.1 mm, vias 0 -> 3
- net TRIG: track 3.68 -> 94.8 mm
- net +14V: track 176.9 -> 258.3 mm, vias 0 -> 2
- net LID: track 10.9 -> 87.7 mm
- net RA4: track 0.00 -> 51.2 mm
- net RG4: track 0.00 -> 34.0 mm
- net RH5: track 5.40 -> 34.0 mm
- net J4-6: track 0.00 -> 28.6 mm
- net RH7: track 0.00 -> 26.5 mm
- net RH6: track 0.00 -> 24.3 mm
- net RE7: track 83.0 -> 58.9 mm, vias 0 -> 1
- net CN1_5V: track 43.6 -> 25.5 mm
- net WDOG_IN: track 8.62 -> 26.5 mm
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- added copper zone on B.Cu, net GND
- added copper zone on F.Cu, net GND
Other:
- board text added: "ATV Control HAT [TFCB]"
- board text added: "BJH 08/15"
